File: power_main/power.kicad_sch (KiCad schematic)
At the start: 82 parts, among them IC1 TPS7A2450DBVR, IC2 TPD4S480RUKR, IC3 CAT24C512WI-GT3, J2 DX07P024AJ1R1500, J3 Conn_02x10_Counter_Clockwise, J4 Conn_02x10_Counter_Clockwise, J5 DX07S024JJ2R1300, J6 DX07S024JJ2R1300, Q1 CSD18543Q3A, Q2 2N7002DW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

Commit message: add missing GPIO_PF small trace refactoring
Connections:
- net GPIO_PF: now also Q9.2 (G), R97.2, R98.2
Other:
- moved on the sheet: C1, C10, C11, C12, C13, C14, C15, C16, C17, C18, C2, C3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
