File: PCB/power_main/power.kicad_sch (KiCad schematic)
At the start: 82 parts, among them IC1 TPS7A2450DBVR, IC2 TPD4S480RUKR, IC3 CAT24C512WI-GT3, J2 DX07P024AJ1R1500, J3 Conn_02x10_Counter_Clockwise, J4 Conn_02x10_Counter_Clockwise, J5 DX07S024JJ2R1300, J6 DX07S024JJ2R1300, Q1 CSD18543Q3A, Q2 2N7002DW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

Commit message: removed POWER_PATH_EN logic add more doku and pictires for context
Parts:
- removed Q2: 2N7002DW, Package_TO_SOT_SMD:SOT-363_SC-70-6, symbol Transistor_FET:Q_Dual_NMOS_S1G1D2S2G2D1
- removed R1, R2: 1.00k, Resistor_SMD:R_0402_1005Metric, symbol Device:R
- IC1: value TPS7A2450DBVR -> TPS7A24
- IC2: value TPD4S480RUKR -> TPD4S480
- IC3: value CAT24C512WI-GT3 -> CAT24C512
- J2: value DX07P024AJ1R1500 -> DX07P024AJ1R1500 - Plug
- J5, J6: value DX07S024JJ2R1300 -> DX07S024JJ2R1300 - Connector
- PS1: value TPSM365R15RDNR -> TPSM365R6
- U1: value TPS26750SRSMR -> TPS26750
Connections:
- net D00 renamed DO0
- no-connect marks 87 -> 88
Other:
- note added: "3V3 LDO - PD IC"
- note added: "5V LDO"
- note added: "DC/DC - 48V/7V"
- note added: "EEPROM"
- note added: "ESP32 Header"
- note added: "Pogo connector - Matrix"
- note added: "Power Delivery (PD) 3.1"
- note added: "Power Output - USB-C"
- note added: "USB C ERP Port Protector"
- note added: "USB-C PD Input"
- moved on the sheet: C1, C10, C11, C12, C13, C14, C15, C16, C17, C18, C19, C2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
